Commit message: feat: camera_frame and sim_unity args

File: kortex_description/robots/kinova.urdf.xacro (robot description, xacro)
@@ -25,4 +25,5 @@
   <xacro:arg name="sim_ignition" default="false" />
   <xacro:arg name="sim_isaac" default="false" />
+  <xacro:arg name="sim_unity" default="false"/>
   <xacro:arg name="gazebo_renderer" default="ogre"/>
   <xacro:arg name="camera_width" default="640"/>
@@ -64,4 +65,25 @@
     <origin xyz="0 0 0" rpy="0 0 0" />  <!-- position robot in the world -->
   </xacro:load_robot>
+  <xacro:if value="$(arg sim_unity)">
+    <joint name="camera_joint" type="fixed">
+      <parent link="world" />
+      <child link="camera_frame" />
+    </joint>
+    <link name="camera_frame">
+      <visual>
+        <origin xyz="0 1 0" rpy="0 0 0"/>
+        <geometry>
+          <box size="0.01 0.01 0.01"/>
+        </geometry>
+      </visual>
+    </link>
+    <sensor name="camera_name" update_rate="20">
+      <parent link="camera_frame"/>
+      <origin xyz="0 0 0" rpy="0 0 0"/>
+      <camera>
+        <image width="640" height="480" hfov="1.5708" format="RGB8" near="0.01" far="50.0"/>
+      </camera>
+    </sensor>
+  </xacro:if>
   <xacro:if value="$(arg sim_gazebo)">
     <!-- Gazebo plugins -->
